File: iteration2/test.kicad_sch (KiCad schematic)
At the start: 95 parts, among them U1 Raspberry_Pi_Pico

Commit message: update layout
Parts:
- D1, D10, D11, D12, D13, D14, D15, D16, D17, D18, D19, D2, D20, D21, D22, D23, D24, D25, D26, D27, D3, D4, D5, D6, D7, D8, D9: footprint ScottoKeebs_Components:Diode_DO-35 -> Diode_SMD:D_SOD-123; symbol ScottoKeebs:Placeholder_Diode -> Device:D_Small
- renumbered LED6 to LED10, LED20 to LED16, LED19 to LED17, LED17 to LED19, LED16 to LED20, LED10 to LED6, LED9 to LED7, LED7 to LED9
Connections:
- net KEY_LEDS: now also U1.29 (GPIO22)
Other:
- moved on the sheet: D1, D10, D11, D12, D13, D14, D15, D16, D17, D18, D19, D2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
